Commit message: urdf wheel

File: src/ugv/src/urdf/leo.urdf (robot description, URDF)
Before this commit: robot leo, 4 links, 3 joints
Links:
- link chassis: geometry collision box size=0.0 0.0 0.0; visual mesh filename=package://ugv/src/meshes/Chassis.dae
- link rocker_left: geometry collision box size=0.0 0.0 0.0; visual mesh filename=package://ugv/src/meshes/Rocker.dae
- link rocker_right: geometry collision box size=0.0 0.0 0.0; visual mesh filename=package://ugv/src/meshes/Rocker.dae
- link wheel_right_front: geometry collision box size=0.0 0.0 0.0; visual mesh filename=package://ugv/src/meshes/WheelB.dae
Joints:
- joint wheel_right_front_joint: axis 0.0 0.0 0.0 -> 0.0 1.0 0.0; limit lower=0.0 upper=0.0 effort=0.0 velocity=0.0 -> lower=0.0 upper=6.28 effort=0.0 velocity=0.01; origin xyz=0.0 0.2 0.0 rpy=0.0 0.0 0.0 -> xyz=0.15 -0.08 -0.09 rpy=0.0 0.0 0.0; type revolute -> continuous

Commit message: urdf complete

File: src/ugv/src/urdf/leo.urdf (robot description, URDF)
Before this commit: robot leo, 4 links, 3 joints
Links:
- added link wheel_left_back, mass 0.0; collision box size=0.0 0.0 0.0; visual mesh filename=package://ugv/src/meshes/WheelA.dae
- added link wheel_left_front, mass 0.0; collision box size=0.0 0.0 0.0; visual mesh filename=package://ugv/src/meshes/WheelA.dae
- added link wheel_right_back, mass 0.0; collision box size=0.0 0.0 0.0; visual mesh filename=package://ugv/src/meshes/WheelB.dae
Joints:
- added joint wheel_left_back_joint: type continuous, parent rocker_left, child wheel_left_back, origin xyz=-0.15 -0.08 -0.09 rpy=0.0 0.0 0.0, axis 0.0 1.0 0.0, limit lower=0.0 upper=6.28 effort=0.0 velocity=0.01
- added joint wheel_left_front_joint: type continuous, parent rocker_left, child wheel_left_front, origin xyz=0.15 -0.08 -0.09 rpy=0.0 0.0 0.0, axis 0.0 1.0 0.0, limit lower=0.0 upper=6.28 effort=0.0 velocity=0.01
- added joint wheel_right_back_joint: type continuous, parent rocker_right, child wheel_right_back, origin xyz=-0.15 -0.08 -0.09 rpy=0.0 0.0 0.0, axis 0.0 1.0 0.0, limit lower=0.0 upper=6.28 effort=0.0 velocity=0.01

Commit message: update

File: src/ugv/src/urdf/leo.urdf (robot description, URDF)
Before this commit: robot leo, 7 links, 6 joints
Links:
- link rocker_left: mass 0.0 -> 1.387336; geometry collision mesh filename=package://ugv/src/meshes/Rocker_outline.stl; visual mesh filename=package://ugv/src/meshes/Rocker.dae
- link rocker_right: mass 0.0 -> 1.387336; geometry collision mesh filename=package://ugv/src/meshes/Rocker_outline.stl; visual mesh filename=package://ugv/src/meshes/Rocker.dae
- link wheel_left_back: mass 0.0 -> 0.283642; geometry collision cylinder length=0.04 radius=0.0625; collision cylinder length=0.07 radius=0.057
- link wheel_left_front: mass 0.0 -> 0.283642; geometry collision cylinder length=0.04 radius=0.0625; collision cylinder length=0.07 radius=0.057
- link wheel_right_back: mass 0.0 -> 0.283642; geometry collision cylinder length=0.04 radius=0.0625; collision cylinder length=0.07 radius=0.057
- link wheel_right_front: mass 0.0 -> 0.283642; geometry collision cylinder length=0.04 radius=0.0625; collision cylinder length=0.07 radius=0.057

Commit message: gazebo

File: src/ugv/src/urdf/leo.urdf (robot description, URDF)
Before this commit: robot leo, 7 links, 6 joints
Joints:
- joint rocker_right_joint: origin xyz=0.003 -0.145 -0.045 rpy=0.0 0.0 0.0 -> xyz=0 0.01346 -0.06506 rpy=0.0 0.0 0.0

Commit message: edit

File: src/ugv/src/urdf/leo.urdf (robot description, URDF)
Before this commit: robot leo, 7 links, 6 joints
Links:
- link wheel_left_back: geometry collision cylinder length=0.04 radius=0.0625; collision cylinder length=0.07 radius=0.057
- link wheel_left_front: geometry collision cylinder length=0.04 radius=0.0625; collision cylinder length=0.07 radius=0.057
Joints:
- joint rocker_right_joint: origin xyz=0 0.01346 -0.06506 rpy=0.0 0.0 0.0 -> xyz=0.003 -0.145 -0.045 rpy=0.0 0.0 0.0
- joint wheel_left_back_joint: axis 0.0 1.0 0.0 -> 0 -1 0; limit lower=0.0 upper=6.28 effort=0.0 velocity=0.01 -> effort=2.0 velocity=6.0; origin xyz=-0.15 -0.08 -0.09 rpy=0.0 0.0 0.0 -> xyz=0.15256 -0.08214 -0.08802 rpy=0 0 0
- joint wheel_left_front_joint: axis 0.0 1.0 0.0 -> 0 -1 0; limit lower=0.0 upper=6.28 effort=0.0 velocity=0.01 -> effort=2.0 velocity=6.0; origin xyz=0.15 -0.08 -0.09 rpy=0.0 0.0 0.0 -> xyz=-0.15256 -0.08214 -0.08802 rpy=0 0 0
- joint wheel_right_back_joint: axis 0.0 1.0 0.0 -> 0 1 0; limit lower=0.0 upper=6.28 effort=0.0 velocity=0.01 -> effort=2.0 velocity=6.0; origin xyz=-0.15 -0.08 -0.09 rpy=0.0 0.0 0.0 -> xyz=-0.15256 -0.08214 -0.08802 rpy=0 0 0
- joint wheel_right_front_joint: limit lower=0.0 upper=6.28 effort=0.0 velocity=0.01 -> effort=2.0 velocity=6.0; origin xyz=0.15 -0.08 -0.09 rpy=0.0 0.0 0.0 -> xyz=0.15256 -0.08214 -0.08802 rpy=0 0 0

Commit message: camera

File: src/ugv/src/urdf/leo.urdf (robot description, URDF)
Before this commit: robot leo, 7 links, 6 joints
Links:
- added link camera_frame
- added link camera_optical_frame
- added link imu_frame
Joints:
- added joint camera_joint: type fixed, parent chassis, child camera_frame, origin xyz=0.0971 0 -0.0427 rpy=0 0.2094 0
- added joint camera_optical_joint: type fixed, parent camera_frame, child camera_optical_frame, origin xyz=0 0 0 rpy=-1.57 0.0 -1.57
- added joint imu_joint: type fixed, parent chassis, child imu_frame, origin xyz=0.0628 -0.0314 -0.0393 rpy=0 0 0
- joint wheel_left_back_joint: type continuous -> revolute
- joint wheel_right_back_joint: type continuous -> revolute

Commit message: camera

File: src/ugv/src/urdf/leo.urdf (robot description, URDF)
Before this commit: robot leo, 10 links, 9 joints
Links:
- added link landing_pad, mass 0.001; collision box size=0.0 0.0 0.0; visual box size=0.3 0.4 0.01
Joints:
- added joint landingPadjoint: type fixed, parent chassis, child landing_pad, origin xyz=0.0 0.0 0.5 rpy=0.0 0.0 0.0, axis 0.0 0.0 0.0, limit lower=0.0 upper=0.0 effort=0.0 velocity=0.0

Commit message: edit

File: src/ugv/src/urdf/leo.urdf (robot description, URDF)
Before this commit: robot leo, 11 links, 10 joints
Joints:
- joint rocker_left_joint: axis 0.0 0.0 0.0 -> 0.0 1.0 0.0; origin xyz=0.003 0.145 -0.045 rpy=0.0 0.0 3.14 -> xyz=0.00263 0.14167 -0.04731 rpy=0.0 0.0 3.14
- joint rocker_right_joint: axis 0.0 0.0 0.0 -> 0.0 1.0 0.0; origin xyz=0.003 -0.145 -0.045 rpy=0.0 0.0 0.0 -> xyz=0.00263 -0.14167 -0.04731 rpy=0.0 0.0 0.0

Commit message: skid drive

File: src/ugv/src/urdf/leo.urdf (robot description, URDF)
Before this commit: robot leo, 11 links, 10 joints
Links:
- link landing_pad: geometry collision box size=0.0 0.0 0.0; visual box size=0.3 0.3 0.01
Joints:
- joint landingPadjoint: axis 0.0 0.0 0.0 -> 1.0 0.0 0.0; origin xyz=0.0 0.0 0.5 rpy=0.0 0.0 0.0 -> xyz=0.0 0.0 0.02 rpy=0.0 0.0 0.0
- joint wheel_left_back_joint: type revolute -> continuous
- joint wheel_right_back_joint: type revolute -> continuous

Commit message: aruco oon top

File: src/ugv/src/urdf/leo.urdf (robot description, URDF)
Before this commit: robot leo, 11 links, 10 joints
Links:
- added link aruco; visual mesh filename=package://ugv/src/meshes/Marker4.dae scale=0.5 0.5 0.5
Joints:
- added joint aruco_joint: type fixed, parent landing_pad, child aruco, origin xyz=0.0 -0.13  0.03 rpy=0.0 0.0 0.0, axis 0.0 0.0 0.0
